File: circuit/VW-R1.sch (KiCad schematic (older format))
At the start: 22 parts, among them J1 PIC16F1938, P1 PICkit3, P2 CONN_02X05, SW1 reset

Commit message: [add] いろいろできるようにコネクタを追加
5ピンコネクタx2.
	・5V/RA3/RA4/RA5/GND
	・5V/RC0/RC1/RC2/GND
Parts:
- added P3, P4: CONN_01X05, Pin_Headers:Pin_Header_Angled_1x05, symbol CONN_01X05
- D1, D2, D3, D4, D5, D6, D7, D8: symbol LED -> LED-RESCUE-VW-R1
Connections:
- net +5V: now also P3.5 (P5), P4.5 (P5)
- net GND: now also P3.1 (P1), P4.1 (P1)
- net at J1.11 (RC0): now also P4.4 (P4)
- net at J1.12 (RC1): now also P4.3 (P3)
- net at J1.13 (RC2): now also P4.2 (P2)
- net at J1.4 (RA2): now also P3.4 (P4)
- net at J1.5 (RA3): now also P3.3 (P3)
- net at J1.6 (RA4): now also P3.2 (P2)
- no-connect marks 13 -> 7
